File: h_bridge_2018.sch (KiCad schematic (older format))
At the start: 12 parts, among them J1 Conn_01x03, J2 alim_puissance_12V, J3 alim_puissance_12V, U1 LMD18200

Commit message: Update h_bridge_2018.sch
Parts:
- removed J3: alim_puissance_12V, symbol @Robot:alim_puissance_12V
- added J?: Conn_01x02, symbol Connector_Generic:Conn_01x02
Connections:
- wire segments 46 -> 36
- no-connect marks 2 -> 0
Changed lines of the file:
@@
 EESchema Schematic File Version 4
-LIBS:schema-cache
 EELAYER 26 0
 EELAYER END
@@
 L Device:C C2
 U 1 1 5C12661E
-P 7250 3050
-F 0 "C2" V 6998 3050 50  0000 C CNN
-F 1 "C" V 7089 3050 50  0000 C CNN
-F 2 "" H 7288 2900 50  0001 C CNN
-F 3 "~" H 7250 3050 50  0001 C CNN
-	1    7250 3050
+P 7400 2500
+F 0 "C2" V 7148 2500 50  0000 C CNN
+F 1 "C" V 7239 2500 50  0000 C CNN
+F 2 "" H 7438 2350 50  0001 C CNN
+F 3 "~" H 7400 2500 50  0001 C CNN
+	1    7400 2500
 	0    1    1    0
 $EndComp
@@
 L Device:C C3
 U 1 1 5C1266DC
-P 8500 3350
-F 0 "C3" V 8248 3350 50  0000 C CNN
-F 1 "C" V 8339 3350 50  0000 C CNN
-F 2 "" H 8538 3200 50  0001 C CNN
-F 3 "~" H 8500 3350 50  0001 C CNN
-	1    8500 3350
-	0    1    1    0
-$EndComp
-$Comp
-L power:GND #PWR02
-U 1 1 5C126D72
-P 6000 1450
-F 0 "#PWR02" H 6000 1200 50  0001 C CNN
-F 1 "GND" H 6005 1277 50  0000 C CNN
-F 2 "" H 6000 1450 50  0001 C CNN
-F 3 "" H 6000 1450 50  0001 C CNN
-	1    6000 1450
-	1    0    0    -1
+P 7250 2750
+F 0 "C3" V 6998 2750 50  0000 C CNN
+F 1 "C" V 7089 2750 50  0000 C CNN
+F 2 "" H 7288 2600 50  0001 C CNN
+F 3 "~" H 7250 2750 50  0001 C CNN
+	1    7250 2750
+	0    1    1    0
 $EndComp
 $Comp
 L Device:R R1
 U 1 1 5C12713F
-P 4050 3100
-F 0 "R1" V 3843 3100 50  0000 C CNN
-F 1 "R" V 3934 3100 50  0000 C CNN
-F 2 "" V 3980 3100 50  0001 C CNN
-F 3 "~" H 4050 3100 50  0001 C CNN
-	1    4050 3100
+P 4950 2800
+F 0 "R1" V 4743 2800 50  0000 C CNN
+F 1 "R" V 4834 2800 50  0000 C CNN
+F 2 "" V 4880 2800 50  0001 C CNN
+F 3 "~" H 4950 2800 50  0001 C CNN
+	1    4950 2800
 	0    1    1    0
 $EndComp
@@
 L Device:R R2
 U 1 1 5C1271CA
-P 4050 2750
-F 0 "R2" V 3843 2750 50  0000 C CNN
-F 1 "R" V 3934 2750 50  0000 C CNN
-F 2 "" V 3980 2750 50  0001 C CNN
-F 3 "~" H 4050 2750 50  0001 C CNN
-	1    4050 2750
+P 5150 2500
+F 0 "R2" V 4943 2500 50  0000 C CNN
+F 1 "R" V 5034 2500 50  0000 C CNN
+F 2 "" V 5080 2500 50  0001 C CNN
+F 3 "~" H 5150 2500 50  0001 C CNN
+	1    5150 2500
 	0    1    1    0
 $EndComp
@@
 L Device:C C1
 U 1 1 5C128A33
-P 5650 3950
-F 0 "C1" H 5765 3996 50  0000 L CNN
-F 1 "C" H 5765 3905 50  0000 L CNN
-F 2 "" H 5688 3800 50  0001 C CNN
-F 3 "~" H 5650 3950 50  0001 C CNN
-	1    5650 3950
-	0    -1   -1   0
+P 5450 2000
+F 0 "C1" H 5565 2046 50  0000 L CNN
+F 1 "C" H 5565 1955 50  0000 L CNN
+F 2 "" H 5488 1850 50  0001 C CNN
+F 3 "~" H 5450 2000 50  0001 C CNN
+	1    5450 2000
+	0    1    1    0
 $EndComp
 $Comp
@@
 	6800 5000 6850 5000
 Wire Wire Line
-	3900 2750 3900 2600
-Wire Wire Line
-	3850 2700 3850 3100
-Wire Wire Line
 	3850 3100 3900 3100
 $Comp
@@
 Wire Wire Line
 	3750 3450 3750 3550
-Wire Wire Line
-	5450 3150 4600 3150
-Wire Wire Line
-	4600 3150 4600 2750
-Wire Wire Line
-	4600 2750 4200 2750
-Wire Wire Line
-	4200 3100 4400 3100
-Wire Wire Line
-	4400 3100 4400 3450
-Wire Wire Line
-	4400 3450 5450 3450
-Wire Wire Line
-	5500 3950 3050 3950
-Wire Wire Line
-	3050 3950 3050 2150
-Wire Wire Line
-	3050 2150 3200 2150
-Wire Wire Line
-	5200 2150 5200 2850
-Wire Wire Line
-	5200 2850 5450 2850
-Wire Wire Line
-	3200 2000 3200 2150
-Connection ~ 3200 2150
-Wire Wire Line
-	3200 2150 5200 2150
-Wire Wire Line
-	3200 2150 3200 4300
-Wire Wire Line
-	3200 4300 2550 4300
-Wire Wire Line
-	2550 4300 2550 1450
-Wire Wire Line
-	2550 1450 6000 1450
-Wire Wire Line
-	6850 3250 7100 3250
-Wire Wire Line
-	7100 3250 7100 3050
-Wire Wire Line
-	6850 3450 8350 3450
-Wire Wire Line
-	8350 3450 8350 3350
-Wire Wire Line
-	8650 3350 8650 3050
-Wire Wire Line
-	6850 3750 8950 3750
-Wire Wire Line
-	8950 3750 8950 3050
-Wire Wire Line
-	8950 3050 8650 3050
 $Comp
 L power:GND #PWR0101
@@
 	1    0    0    -1
 $EndComp
-Wire Wire Line
-	3600 2600 3900 2600
-Wire Wire Line
-	3600 2700 3850 2700
-$Comp
-L @Robot:alim_puissance_12V J3
-U 1 1 5C12B971
-P 8250 2850
-F 0 "J3" H 8194 2533 50  0000 C CNN
-F 1 "alim_puissance_12V" H 8194 2624 50  0000 C CNN
-F 2 "" H 8250 2850 50  0001 C CNN
-F 3 "~" H 8250 2850 50  0001 C CNN
-	1    8250 2850
-	1    0    0    1
-$EndComp
-Wire Wire Line
-	6850 2950 7550 2950
-Wire Wire Line
-	7400 3050 7550 3050
-Wire Wire Line
-	7550 3050 7550 2950
 $Comp
 L @Robot:alim_puissance_12V J2
@@
 Wire Wire Line
 	3750 2800 3600 2800
-Wire Wire Line
-	6150 2250 6150 2000
-Wire Wire Line
-	6150 2000 3200 2000
 $Comp
 L Driver_Motor:LMD18200 U1
 U 1 1 5C126582
-P 6150 3150
-F 0 "U1" H 6150 2072 50  0000 C CNN
-F 1 "LMD18200" H 6150 2163 50  0000 C CNN
-F 2 "Package_TO_SOT_THT:TO-220-11_P3.4x5.08mm_StaggerOdd_Lead4.85mm_Vertical" H 4700 1800 50  0001 L CNN
-F 3 "http://www.ti.com/lit/ds/symlink/lmd18200.pdf" H 6050 3150 50  0001 C CNN
-	1    6150 3150
-	1    0    0    1
-$EndComp
-Wire Wire Line
-	5800 3950 6150 3950
-NoConn ~ 6850 2650
-NoConn ~ 6850 2750
-Wire Wire Line
-	7550 2750 7550 2950
-Connection ~ 7550 2950
+P 6300 2800
+F 0 "U1" H 6300 1722 50  0000 C CNN
+F 1 "LMD18200" H 6300 1813 50  0000 C CNN
+F 2 "Package_TO_SOT_THT:TO-220-11_P3.4x5.08mm_StaggerOdd_Lead4.85mm_Vertical" H 4850 1450 50  0001 L CNN
+F 3 "http://www.ti.com/lit/ds/symlink/lmd18200.pdf" H 6200 2800 50  0001 C CNN
+	1    6300 2800
+	1    0    0    -1
+$EndComp
+Wire Wire Line
+	5950 3600 6300 3600
+$Comp
+L Connector_Generic:Conn_01x02 J?
+U 1 1 5C1BFABE
+P 8000 2500
+F 0 "J?" H 8080 2492 50  0000 L CNN
+F 1 "Conn_01x02" H 8080 2401 50  0000 L CNN
+F 2 "" H 8000 2500 50  0001 C CNN
+F 3 "~" H 8000 2500 50  0001 C CNN
+	1    8000 2500
+	1    0    0    -1
+$EndComp
+Wire Wire Line
+	7000 2500 7250 2500
+Wire Wire Line
+	7550 2500 7650 2500
+Wire Wire Line
+	7000 2200 7650 2200
+Wire Wire Line
+	7650 2200 7650 2500
+Connection ~ 7650 2500
+Wire Wire Line
+	7650 2500 7800 2500
+Wire Wire Line
+	7000 3000 7800 3000
+Wire Wire Line
+	7800 3000 7800 2750
+Wire Wire Line
+	7000 2700 7100 2700
+Wire Wire Line
+	7100 2700 7100 2750
+Wire Wire Line
+	7400 2750 7800 2750
+Connection ~ 7800 2750
+Wire Wire Line
+	7800 2750 7800 2600
+Wire Wire Line
+	6300 2000 5600 2000
+Wire Wire Line
+	5600 2500 5300 2500
+Wire Wire Line
+	5000 2500 3600 2500
+Wire Wire Line
+	3600 2500 3600 2600
+Wire Wire Line
+	5600 2800 5100 2800
+Wire Wire Line
+	4800 2800 4800 2700
+Wire Wire Line
+	4800 2700 3600 2700
+Wire Wire Line
+	5600 3100 5500 3100
+Wire Wire Line
+	5300 3100 5300 2500
+Connection ~ 5300 2500
+Wire Wire Line
+	5300 2500 5300 2000
+Wire Wire Line
+	6300 3700 5500 3700
+Wire Wire Line
+	5500 3700 5500 3100
+Connection ~ 5500 3100
+Wire Wire Line
+	5500 3100 5300 3100
+$Comp
+L power:GND #PWR?
+U 1 1 5C1D359F
+P 5500 2650
+F 0 "#PWR?" H 5500 2400 50  0001 C CNN
+F 1 "GND" H 5505 2477 50  0000 C CNN
+F 2 "" H 5500 2650 50  0001 C CNN
+F 3 "" H 5500 2650 50  0001 C CNN
+	1    5500 2650
+	-1   0    0    1
+$EndComp
+Wire Wire Line
+	5500 3100 5500 2650
 $EndSCHEMATC

Commit message: Update h_bridge_2018.sch
Parts:
- D1: value LED -> LED_3MM ROUGE
- J1: value Conn_01x03 -> PWM_IN
- J2: value alim_puissance_12V -> _P
- J3: renamed from J?; value Conn_01x02 -> U$4
Connections:
- wire segments 36 -> 34
- no-connect marks 0 -> 2
Changed lines of the file:
@@
 EESchema Schematic File Version 4
+LIBS:h_bridge_2018-cache
 EELAYER 26 0
 EELAYER END
@@
 L Device:R R2
 U 1 1 5C1271CA
-P 5150 2500
-F 0 "R2" V 4943 2500 50  0000 C CNN
-F 1 "R" V 5034 2500 50  0000 C CNN
-F 2 "" V 5080 2500 50  0001 C CNN
-F 3 "~" H 5150 2500 50  0001 C CNN
-	1    5150 2500
+P 4800 2500
+F 0 "R2" V 4593 2500 50  0000 C CNN
+F 1 "R" V 4684 2500 50  0000 C CNN
+F 2 "" V 4730 2500 50  0001 C CNN
+F 3 "~" H 4800 2500 50  0001 C CNN
+	1    4800 2500
 	0    1    1    0
 $EndComp
@@
 P 6700 4650
 F 0 "D1" H 6692 4395 50  0000 C CNN
-F 1 "LED" H 6692 4486 50  0000 C CNN
+F 1 "LED_3MM ROUGE" H 6692 4486 50  0000 C CNN
 F 2 "" H 6700 4650 50  0001 C CNN
 F 3 "~" H 6700 4650 50  0001 C CNN
@@
 Wire Wire Line
 	6800 5000 6850 5000
-Wire Wire Line
-	3850 3100 3900 3100
 $Comp
 L Device:R R4
@@
 P 7050 4900
 F 0 "J2" H 7179 4900 50  0000 L CNN
-F 1 "alim_puissance_12V" H 7179 4809 50  0000 L CNN
+F 1 "_P" H 7179 4809 50  0000 L CNN
 F 2 "" H 7050 4900 50  0001 C CNN
 F 3 "~" H 7050 4900 50  0001 C CNN
@@
 P 3400 2700
 F 0 "J1" H 3320 3017 50  0000 C CNN
-F 1 "Conn_01x03" H 3320 2926 50  0000 C CNN
+F 1 "PWM_IN" H 3320 2926 50  0000 C CNN
 F 2 "" H 3400 2700 50  0001 C CNN
 F 3 "~" H 3400 2700 50  0001 C CNN
@@
 	5950 3600 6300 3600
 $Comp
-L Connector_Generic:Conn_01x02 J?
+L Connector_Generic:Conn_01x02 J3
 U 1 1 5C1BFABE
 P 8000 2500
-F 0 "J?" H 8080 2492 50  0000 L CNN
-F 1 "Conn_01x02" H 8080 2401 50  0000 L CNN
+F 0 "J3" H 8080 2492 50  0000 L CNN
+F 1 "U$4" H 8080 2401 50  0000 L CNN
 F 2 "" H 8000 2500 50  0001 C CNN
 F 3 "~" H 8000 2500 50  0001 C CNN
@@
 	6300 2000 5600 2000
 Wire Wire Line
-	5600 2500 5300 2500
-Wire Wire Line
-	5000 2500 3600 2500
-Wire Wire Line
 	3600 2500 3600 2600
 Wire Wire Line
@@
 Wire Wire Line
 	5600 3100 5500 3100
-Wire Wire Line
-	5300 3100 5300 2500
-Connection ~ 5300 2500
-Wire Wire Line
-	5300 2500 5300 2000
 Wire Wire Line
 	6300 3700 5500 3700
@@
 	5500 3100 5300 3100
 $Comp
-L power:GND #PWR?
+L power:GND #PWR0102
 U 1 1 5C1D359F
 P 5500 2650
-F 0 "#PWR?" H 5500 2400 50  0001 C CNN
+F 0 "#PWR0102" H 5500 2400 50  0001 C CNN
 F 1 "GND" H 5505 2477 50  0000 C CNN
 F 2 "" H 5500 2650 50  0001 C CNN
@@
 Wire Wire Line
 	5500 3100 5500 2650
+NoConn ~ 7000 3300
+NoConn ~ 7000 3200
+$Comp
+L power:PWR_FLAG #FLG?
+U 1 1 5C1BE6C2
+P 7650 4900
+F 0 "#FLG?" H 7650 4975 50  0001 C CNN
+F 1 "PWR_FLAG" H 7650 5074 50  0000 C CNN
+F 2 "" H 7650 4900 50  0001 C CNN
+F 3 "~" H 7650 4900 50  0001 C CNN
+	1    7650 4900
+	1    0    0    -1
+$EndComp
+Wire Wire Line
+	5600 2500 4950 2500
+Wire Wire Line
+	4650 2500 3600 2500
+Wire Wire Line
+	5300 3100 5300 2000
 $EndSCHEMATC

Commit message: Update h_bridge_2018.sch
Parts:
- removed J2: _P, symbol @Robot:alim_puissance_12V
- added J2: In_Puissance, symbol Connector_Generic:Conn_01x02
Connections:
- net labels added: VS
- wire segments 34 -> 36
Changed lines of the file:
@@
 	6550 4650 6350 4650
 Wire Wire Line
-	6050 4650 6050 5050
-Wire Wire Line
-	6050 5050 6800 5050
-Wire Wire Line
-	6800 5050 6800 5000
-Wire Wire Line
-	6800 5000 6850 5000
+	6050 4650 6050 5000
 $Comp
 L Device:R R4
@@
 F 3 "" H 3750 3550 50  0001 C CNN
 	1    3750 3550
-	1    0    0    -1
-$EndComp
-$Comp
-L @Robot:alim_puissance_12V J2
-U 1 1 5C130494
-P 7050 4900
-F 0 "J2" H 7179 4900 50  0000 L CNN
-F 1 "_P" H 7179 4809 50  0000 L CNN
-F 2 "" H 7050 4900 50  0001 C CNN
-F 3 "~" H 7050 4900 50  0001 C CNN
-	1    7050 4900
 	1    0    0    -1
 $EndComp
@@
 NoConn ~ 7000 3300
 NoConn ~ 7000 3200
-$Comp
-L power:PWR_FLAG #FLG?
-U 1 1 5C1BE6C2
-P 7650 4900
-F 0 "#FLG?" H 7650 4975 50  0001 C CNN
-F 1 "PWR_FLAG" H 7650 5074 50  0000 C CNN
-F 2 "" H 7650 4900 50  0001 C CNN
-F 3 "~" H 7650 4900 50  0001 C CNN
-	1    7650 4900
-	1    0    0    -1
-$EndComp
 Wire Wire Line
 	5600 2500 4950 2500
@@
 Wire Wire Line
 	5300 3100 5300 2000
+Text Label 6050 4900 0    50   ~ 0
+VS
+Text Label 5800 2000 0    50   ~ 0
+VS
+$Comp
+L power:PWR_FLAG #FLG0101
+U 1 1 5C1C3E4F
+P 6900 5000
+F 0 "#FLG0101" H 6900 5075 50  0001 C CNN
+F 1 "PWR_FLAG" H 6900 5174 50  0000 C CNN
+F 2 "" H 6900 5000 50  0001 C CNN
+F 3 "~" H 6900 5000 50  0001 C CNN
+	1    6900 5000
+	-1   0    0    1
+$EndComp
+$Comp
+L power:PWR_FLAG #FLG0102
+U 1 1 5C1C40EA
+P 6900 4900
+F 0 "#FLG0102" H 6900 4975 50  0001 C CNN
+F 1 "PWR_FLAG" H 6900 5074 50  0000 C CNN
+F 2 "" H 6900 4900 50  0001 C CNN
+F 3 "~" H 6900 4900 50  0001 C CNN
+	1    6900 4900
+	1    0    0    -1
+$EndComp
+Wire Wire Line
+	6850 4900 6900 4900
+Wire Wire Line
+	6050 5000 6900 5000
+Connection ~ 6900 5000
+Connection ~ 6900 4900
+Wire Wire Line
+	6900 5000 7100 5000
+Wire Wire Line
+	6900 4900 7050 4900
+$Comp
+L power:GND #PWR0103
+U 1 1 5C1CB26F
+P 7050 4900
+F 0 "#PWR0103" H 7050 4650 50  0001 C CNN
+F 1 "GND" H 7055 4727 50  0000 C CNN
+F 2 "" H 7050 4900 50  0001 C CNN
+F 3 "" H 7050 4900 50  0001 C CNN
+	1    7050 4900
+	-1   0    0    1
+$EndComp
+Connection ~ 7050 4900
+Wire Wire Line
+	7050 4900 7100 4900
+$Comp
+L Connector_Generic:Conn_01x02 J2
+U 1 1 5C1CBBA5
+P 7300 4900
+F 0 "J2" H 7380 4892 50  0000 L CNN
+F 1 "In_Puissance" H 7380 4801 50  0000 L CNN
+F 2 "" H 7300 4900 50  0001 C CNN
+F 3 "~" H 7300 4900 50  0001 C CNN
+	1    7300 4900
+	1    0    0    -1
+$EndComp
 $EndSCHEMATC

Commit message: Update h_bridge_2018.sch
Parts:
- C1: value C -> 470uF
Connections:
- wire segments 36 -> 38
Changed lines of the file:
@@
 L Device:C C1
 U 1 1 5C128A33
-P 5450 2000
-F 0 "C1" H 5565 2046 50  0000 L CNN
-F 1 "C" H 5565 1955 50  0000 L CNN
-F 2 "" H 5488 1850 50  0001 C CNN
-F 3 "~" H 5450 2000 50  0001 C CNN
-	1    5450 2000
+P 6500 4250
+F 0 "C1" H 6615 4296 50  0000 L CNN
+F 1 "470uF" H 6615 4205 50  0000 L CNN
+F 2 "" H 6538 4100 50  0001 C CNN
+F 3 "~" H 6500 4250 50  0001 C CNN
+	1    6500 4250
 	0    1    1    0
 $EndComp
@@
 	7800 2750 7800 2600
 Wire Wire Line
-	6300 2000 5600 2000
-Wire Wire Line
 	3600 2500 3600 2600
 Wire Wire Line
@@
 Wire Wire Line
 	5500 3700 5500 3100
-Connection ~ 5500 3100
-Wire Wire Line
-	5500 3100 5300 3100
 $Comp
 L power:GND #PWR0102
 U 1 1 5C1D359F
-P 5500 2650
-F 0 "#PWR0102" H 5500 2400 50  0001 C CNN
-F 1 "GND" H 5505 2477 50  0000 C CNN
-F 2 "" H 5500 2650 50  0001 C CNN
-F 3 "" H 5500 2650 50  0001 C CNN
-	1    5500 2650
-	-1   0    0    1
-$EndComp
-Wire Wire Line
-	5500 3100 5500 2650
+P 5350 3100
+F 0 "#PWR0102" H 5350 2850 50  0001 C CNN
+F 1 "GND" H 5355 2927 50  0000 C CNN
+F 2 "" H 5350 3100 50  0001 C CNN
+F 3 "" H 5350 3100 50  0001 C CNN
+	1    5350 3100
+	0    1    1    0
+$EndComp
 NoConn ~ 7000 3300
 NoConn ~ 7000 3200
@@
 Wire Wire Line
 	4650 2500 3600 2500
-Wire Wire Line
-	5300 3100 5300 2000
 Text Label 6050 4900 0    50   ~ 0
 VS
-Text Label 5800 2000 0    50   ~ 0
+Text Label 6300 1850 0    50   ~ 0
 VS
 $Comp
@@
 	1    0    0    -1
 $EndComp
+Wire Wire Line
+	6050 4650 6050 4250
+Wire Wire Line
+	6050 4250 6350 4250
+Connection ~ 6050 4650
+Wire Wire Line
+	6650 4250 6850 4250
+Wire Wire Line
+	6850 4250 6850 4650
+Connection ~ 6850 4650
+Wire Wire Line
+	5500 3100 5350 3100
+Connection ~ 5500 3100
+Wire Wire Line
+	6300 1850 6300 2000
 $EndSCHEMATC

Commit message: Update h_bridge_2018.sch
Parts:
- C1: footprint (none) -> Capacitor_THT:C_Radial_D10.0mm_H20.0mm_P5.00mm
Changed lines of the file:
@@
 F 0 "C1" H 6615 4296 50  0000 L CNN
 F 1 "470uF" H 6615 4205 50  0000 L CNN
-F 2 "" H 6538 4100 50  0001 C CNN
+F 2 "Capacitor_THT:C_Radial_D10.0mm_H20.0mm_P5.00mm" H 6538 4100 50  0001 C CNN
 F 3 "~" H 6500 4250 50  0001 C CNN
 	1    6500 4250
